File: hardware/design/GameOnSpinner/GameOnSpinner.sch (KiCad schematic (older format))
At the start: 10 parts, among them IC1 A1302KLHLT-T, IC2 A1302KLHLT-T, IC3 A1302KLHLT-T, IC4 A1302KLHLT-T, IC5 A1302KLHLT-T, IC6 A1302KLHLT-T, IC7 A1302KLHLT-T, IC8 A1302KLHLT-T, P1 CONN_01X15, P2 CONN_01X15

Commit message: Add bluetooth board.
Parts:
- added P?: CONN_01X06, symbol CONN_01X06
Connections:
- net at P1.2 (P2): now also P?.5 (P5)
- net at P2.4 (P4): now also P?.4 (P4)
- net at P2.5 (P5): now also P?.2 (P2)
- net at P2.6 (P6): now also P?.3 (P3)
- no-connect marks 20 -> 18
Changed lines of the file:
@@
 LIBS:valves
 LIBS:sensors
+LIBS:GameOnSpinner-cache
 EELAYER 25 0
 EELAYER END
@@
 $EndComp
 $Comp
-L CONN_01X15 P2
-U 1 1 5848B2B9
-P 4750 6300
-F 0 "P2" H 4750 7100 50  0000 C CNN
-F 1 "CONN_01X15" V 4850 6300 50  0000 C CNN
-F 2 "Socket_Strips:Socket_Strip_Straight_1x15" H 4750 6300 50  0001 C CNN
-F 3 "" H 4750 6300 50  0000 C CNN
-	1    4750 6300
-	0    -1   -1   0
-$EndComp
-Wire Wire Line
-	1000 3200 9150 3200
-Wire Wire Line
-	1700 5400 1700 3950
-Wire Wire Line
-	4450 5400 1700 5400
-Wire Wire Line
-	4450 5750 4450 5400
-Wire Wire Line
-	2800 5300 2800 3950
-Wire Wire Line
-	4550 5300 2800 5300
-Wire Wire Line
-	4550 5750 4550 5300
-Wire Wire Line
-	3950 5200 3950 4000
-Wire Wire Line
-	4650 5200 3950 5200
-Wire Wire Line
-	4650 5750 4650 5200
-Wire Wire Line
-	4750 5200 4750 5750
-Wire Wire Line
-	5150 5200 4750 5200
-Wire Wire Line
-	5150 4000 5150 5200
-Wire Wire Line
-	4850 5300 4850 5750
-Wire Wire Line
-	6250 5300 4850 5300
-Wire Wire Line
-	6250 4000 6250 5300
-Wire Wire Line
-	7400 5400 7400 4000
-Wire Wire Line
-	4950 5400 7400 5400
-Wire Wire Line
-	4950 5750 4950 5400
-Wire Wire Line
-	5050 5500 5050 5750
-Wire Wire Line
-	8500 5500 5050 5500
-Wire Wire Line
-	8500 4000 8500 5500
-Wire Wire Line
-	9650 4000 9550 4000
-Wire Wire Line
-	9650 5600 9650 4000
-Wire Wire Line
-	5150 5600 9650 5600
-Wire Wire Line
-	5150 5750 5150 5600
-Wire Wire Line
-	1300 3200 1300 3550
-Connection ~ 9150 3200
-Wire Wire Line
-	9150 3200 9150 3600
-Connection ~ 8100 3200
-Wire Wire Line
-	8100 3600 8100 3200
-Connection ~ 5850 3200
-Wire Wire Line
-	5850 3600 5850 3200
-Connection ~ 7000 3200
-Wire Wire Line
-	7000 3600 7000 3200
-Connection ~ 4750 3200
-Wire Wire Line
-	4750 3600 4750 3200
-Connection ~ 3550 3200
-Wire Wire Line
-	3550 3600 3550 3200
-Connection ~ 2400 3200
-Wire Wire Line
-	2400 3550 2400 3200
-Connection ~ 9150 4850
-Connection ~ 8100 4850
-Wire Wire Line
-	8100 4400 8100 4850
-Connection ~ 7000 4850
-Wire Wire Line
-	7000 4400 7000 4850
-Connection ~ 5850 4850
-Wire Wire Line
-	5850 4400 5850 4850
-Connection ~ 4750 4850
-Wire Wire Line
-	4750 4400 4750 4850
-Connection ~ 3550 4850
-Wire Wire Line
-	3550 4400 3550 4850
-Connection ~ 2400 4850
-Wire Wire Line
-	2400 4350 2400 4850
-Wire Wire Line
-	9150 4400 9150 4850
-Wire Wire Line
-	1300 4350 1300 5600
-Wire Wire Line
-	4350 5750 4350 5500
-Wire Wire Line
-	4350 5500 1000 5500
-Wire Wire Line
-	1000 5500 1000 3200
-Connection ~ 1300 3200
-Wire Wire Line
-	9150 4850 1300 4850
-Wire Wire Line
-	4150 5750 4150 5600
-Wire Wire Line
-	4150 5600 1300 5600
-Connection ~ 1300 4850
-$Comp
 L PWR_FLAG #FLG01
 U 1 1 5848C54D
@@
 	1    0    0    -1
 $EndComp
-Wire Wire Line
-	1050 3150 1050 3200
-Connection ~ 1050 3200
 $Comp
 L PWR_FLAG #FLG02
@@
 	-1   0    0    1
 $EndComp
-Wire Wire Line
-	1350 5750 1350 5600
-Connection ~ 1350 5600
 NoConn ~ 5250 5750
-NoConn ~ 5350 5750
 NoConn ~ 5450 5750
 NoConn ~ 5450 6500
@@
 NoConn ~ 4750 6500
 NoConn ~ 4650 6500
-NoConn ~ 4550 6500
-NoConn ~ 4450 6500
-NoConn ~ 4350 6500
 NoConn ~ 4250 6500
 NoConn ~ 4150 6500
@@
 NoConn ~ 4050 5750
 NoConn ~ 4250 5750
+$Comp
+L CONN_01X06 P?
+U 1 1 5849B8D1
+P 3050 6300
+F 0 "P?" H 3050 6650 50  0000 C CNN
+F 1 "CONN_01X06" V 3150 6300 50  0000 C CNN
+F 2 "" H 3050 6300 50  0000 C CNN
+F 3 "" H 3050 6300 50  0000 C CNN
+	1    3050 6300
+	0    -1   -1   0
+$EndComp
+NoConn ~ 3300 6500
+NoConn ~ 2800 6500
+Wire Wire Line
+	1000 3200 9150 3200
+Wire Wire Line
+	1700 5400 1700 3950
+Wire Wire Line
+	4450 5400 1700 5400
+Wire Wire Line
+	4450 5750 4450 5400
+Wire Wire Line
+	2800 5300 2800 3950
+Wire Wire Line
+	4550 5300 2800 5300
+Wire Wire Line
+	4550 5750 4550 5300
+Wire Wire Line
+	3950 5200 3950 4000
+Wire Wire Line
+	4650 5200 3950 5200
+Wire Wire Line
+	4650 5750 4650 5200
+Wire Wire Line
+	4750 5200 4750 5750
+Wire Wire Line
+	5150 5200 4750 5200
+Wire Wire Line
+	5150 4000 5150 5200
+Wire Wire Line
+	4850 5300 4850 5750
+Wire Wire Line
+	6250 5300 4850 5300
+Wire Wire Line
+	6250 4000 6250 5300
+Wire Wire Line
+	7400 5400 7400 4000
+Wire Wire Line
+	4950 5400 7400 5400
+Wire Wire Line
+	4950 5750 4950 5400
+Wire Wire Line
+	5050 5500 5050 5750
+Wire Wire Line
+	8500 5500 5050 5500
+Wire Wire Line
+	8500 4000 8500 5500
+Wire Wire Line
+	9650 4000 9550 4000
+Wire Wire Line
+	9650 5600 9650 4000
+Wire Wire Line
+	5150 5600 9650 5600
+Wire Wire Line
+	5150 5750 5150 5600
+Wire Wire Line
+	1300 3200 1300 3550
+Connection ~ 9150 3200
+Wire Wire Line
+	9150 3200 9150 3600
+Connection ~ 8100 3200
+Wire Wire Line
+	8100 3600 8100 3200
+Connection ~ 5850 3200
+Wire Wire Line
+	5850 3600 5850 3200
+Connection ~ 7000 3200
+Wire Wire Line
+	7000 3600 7000 3200
+Connection ~ 4750 3200
+Wire Wire Line
+	4750 3600 4750 3200
+Connection ~ 3550 3200
+Wire Wire Line
+	3550 3600 3550 3200
+Connection ~ 2400 3200
+Wire Wire Line
+	2400 3550 2400 3200
+Connection ~ 9150 4850
+Connection ~ 8100 4850
+Wire Wire Line
+	8100 4400 8100 4850
+Connection ~ 7000 4850
+Wire Wire Line
+	7000 4400 7000 4850
+Connection ~ 5850 4850
+Wire Wire Line
+	5850 4400 5850 4850
+Connection ~ 4750 4850
+Wire Wire Line
+	4750 4400 4750 4850
+Connection ~ 3550 4850
+Wire Wire Line
+	3550 4400 3550 4850
+Connection ~ 2400 4850
+Wire Wire Line
+	2400 4350 2400 4850
+Wire Wire Line
+	9150 4400 9150 4850
+Wire Wire Line
+	1300 4350 1300 5600
+Wire Wire Line
+	4350 5750 4350 5500
+Wire Wire Line
+	4350 5500 1000 5500
+Wire Wire Line
+	1000 5500 1000 3200
+Connection ~ 1300 3200
+Wire Wire Line
+	9150 4850 1300 4850
+Wire Wire Line
+	4150 5750 4150 5600
+Wire Wire Line
+	4150 5600 1300 5600
+Connection ~ 1300 4850
+Wire Wire Line
+	1050 3150 1050 3200
+Connection ~ 1050 3200
+Wire Wire Line
+	1350 5750 1350 5600
+Connection ~ 1350 5600
+Wire Wire Line
+	3200 6500 3200 6600
+Wire Wire Line
+	3200 6600 5750 6600
+Wire Wire Line
+	5750 6600 5750 5700
+Wire Wire Line
+	5750 5700 5350 5700
+Wire Wire Line
+	5350 5700 5350 5750
+Wire Wire Line
+	4350 6500 4350 6700
+Wire Wire Line
+	4350 6700 3100 6700
+Wire Wire Line
+	3100 6700 3100 6500
+Wire Wire Line
+	3000 6500 3000 6800
+Wire Wire Line
+	3000 6800 4550 6800
+$Comp
+L CONN_01X15 P2
+U 1 1 5848B2B9
+P 4750 6300
+F 0 "P2" H 4750 7100 50  0000 C CNN
+F 1 "CONN_01X15" V 4850 6300 50  0000 C CNN
+F 2 "Socket_Strips:Socket_Strip_Straight_1x15" H 4750 6300 50  0001 C CNN
+F 3 "" H 4750 6300 50  0000 C CNN
+	1    4750 6300
+	0    -1   -1   0
+$EndComp
+Wire Wire Line
+	4550 6800 4550 6500
+Wire Wire Line
+	4450 6500 4450 6900
+Wire Wire Line
+	4450 6900 2900 6900
+Wire Wire Line
+	2900 6900 2900 6500
 $EndSCHEMATC
